Commit message: add dynamic obstacle&debug line_follower

File: car_sim/akm_description/urdf/ai_akm/aiakm_rplidar.xacro (robot description, xacro)
@@ -6,5 +6,5 @@
             <box_inertial_matrix  m="0.001" w="0.001" h="0.001" d="0.001"/>
             <visual>
-                <origin xyz=" 0 0 0" rpy="0 0 0" />
+                <origin xyz=" 0 0 -0.07 " rpy="0 0 0" />
                 <geometry>
                     <!--add rplidar mesh-->

File: car_sim/akm_description/urdf/ai_akm/aiakm_transmission.xacro (robot description, xacro)
@@ -8,5 +8,5 @@
     <xacro:macro name="wheel_transmission" params="LR FR">
     <gazebo reference="${LR}_${FR}_wheel_link">
-        <material>Gazebo/GreenTransparent</material>
+        <material>Gazebo/Black</material>
         <mu1>1</mu1>
         <mu2>1</mu2>
